Commit message: added SMARC FLS sonar to the rexrov robot description (default)

File: uuv_descriptions/urdf/rexrov_sensors_fls.xacro (robot description, xacro)
@@ -54,18 +54,3 @@
     parent_link="${namespace}/base_link"
     inertial_reference_frame="${inertial_reference_frame}" />
-  <!-- Mount FLS. -->
-  <xacro:forward_looking_sonar
-      namespace="${namespace}"
-      suffix=""
-      parent_link="${namespace}/base_link"
-      topic="fls_sonar"
-      mass="0.1"
-      update_rate="10"
-      samples="512"
-      fov="1.22173"
-      width="512"
-      height="1024" >
-      <inertia ixx="0.00001" ixy="0.0" ixz="0.0" iyy="0.00001" iyz="0.0" izz="0.00001" />
-      <origin xyz="1.3 0 -0.7" rpy="0 0.7853 0" />
-  </xacro:forward_looking_sonar>
 </robot>

File: uuv_sensor_plugins/uuv_sensor_ros_plugins/urdf/sonar_snippets.xacro (robot description, xacro)
@@ -152,7 +152,5 @@
   </gazebo>
   </xacro:macro>
-  <xacro:macro name="forward_looking_sonar"
-    params="namespace suffix parent_link topic mass update_rate
-      samples fov width height *inertia *origin">
+  <xacro:macro name="forward_looking_sonar" params="namespace suffix parent_link topic mass update_rate samples fov width height *inertia *origin">
     <!-- Sensor link -->
     <link name="${namespace}/forward_sonar${suffix}_link">
