Commit message: x,y,z coords of every point in the sonar image now published on /rexrov/depth/image_raw_depth_raw_sonar topic, removed speckle noise (should make it tunable)

File: uuv_descriptions/urdf/rexrov_sensors.xacro (robot description, xacro)
@@ -67,5 +67,5 @@
       height="400" >
       <inertia ixx="0.00001" ixy="0.0" ixz="0.0" iyy="0.00001" iyz="0.0" izz="0.00001" />
-      <origin xyz="1.3 0 -0.7" rpy="0 0.7853 0" />
+      <origin xyz="1.3 0 -0.7" rpy="0 0.4235987 0" />
   </xacro:forward_looking_sonar>
 </robot>

Commit message: cleaning up

File: uuv_descriptions/urdf/rexrov_sensors.xacro (robot description, xacro)
@@ -38,13 +38,13 @@
   </xacro:default_imu_macro>
   <!-- Mount a camera -->
-  <xacro:default_camera namespace="${namespace}" parent_link="${namespace}/base_link" suffix="">
-    <origin xyz="1.15 0 0.4" rpy="0 0.6 0"/>
-  </xacro:default_camera>
-  <xacro:default_camera namespace="${namespace}" parent_link="${namespace}/base_link" suffix="right">
-    <origin xyz="1.15 -0.63 0.4" rpy="0 0.6 0.4"/>
-  </xacro:default_camera>
-  <xacro:default_camera namespace="${namespace}" parent_link="${namespace}/base_link" suffix="left">
-    <origin xyz="1.15 0.63 0.4" rpy="0 0.6 -0.4"/>
-  </xacro:default_camera>
+  <!--<xacro:default_camera namespace="${namespace}" parent_link="${namespace}/base_link" suffix="">-->
+    <!--<origin xyz="1.15 0 0.4" rpy="0 0.6 0"/>-->
+  <!--</xacro:default_camera>-->
+  <!--<xacro:default_camera namespace="${namespace}" parent_link="${namespace}/base_link" suffix="right">-->
+    <!--<origin xyz="1.15 -0.63 0.4" rpy="0 0.6 0.4"/>-->
+  <!--</xacro:default_camera>-->
+  <!--<xacro:default_camera namespace="${namespace}" parent_link="${namespace}/base_link" suffix="left">-->
+    <!--<origin xyz="1.15 0.63 0.4" rpy="0 0.6 -0.4"/>-->
+  <!--</xacro:default_camera>-->
   <!-- Mount a GPS. -->
   <xacro:default_gps namespace="${namespace}" parent_link="${namespace}/base_link" />
@@ -55,4 +55,7 @@
     inertial_reference_frame="${inertial_reference_frame}" />
   <!-- Mount FLS. -->
+  <!--fov="1.22173"-->
+  <!--width="512"-->
+  <!--height="400"-->
   <xacro:forward_looking_sonar
       namespace="${namespace}"
@@ -61,11 +64,12 @@
       topic="fls_sonar"
       mass="0.1"
-      update_rate="10"
+      update_rate="5"
       samples="512"
-      fov="1.22173"
+      fov="0.8726"
       width="512"
-      height="400" >
+      height="115" >
       <inertia ixx="0.00001" ixy="0.0" ixz="0.0" iyy="0.00001" iyz="0.0" izz="0.00001" />
-      <origin xyz="1.3 0 -0.7" rpy="0 0.4235987 0" />
+      <!--<origin xyz="1.3 0 -0.7" rpy="0 0.4235987 0" />-->
+      <origin xyz="1.3 0 -0.7" rpy="0 0 0" />
   </xacro:forward_looking_sonar>
 </robot>
